File: EAGLE/Motherboard.brd (EAGLE design)
At the start: 60.9 x 51.7 mm, 21 parts, among them T1 BC337

Commit message: Got the basic arduino stuff to work
Routing:
- net VCC: track 133.5 -> 123.1 mm
- net D13: track 47.5 -> 54.7 mm, vias 2 -> 0
- net TX: track 6.88 -> 13.8 mm, vias 2 -> 0
- net RX: track 10.5 -> 16.8 mm, vias 2 -> 0
- added copper zone on layer 1, net GND
